File: E-P-099-R2.5.brd (EAGLE design)
At the start: 100 x 80 mm, 86 parts, among them J1 AVR_ISP

Commit message: update
Parts:
- C10: value 18fp -> (none)
- C7, C8, C9: value 18pf -> (none)
Changed lines of the file:
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@@
 <?xml version="1.0" encoding="utf-8"?>
 <!DOCTYPE eagle SYSTEM "eagle.dtd">
-<eagle version="7.5.0">
+<eagle version="7.4.0">
 <drawing>
 <settings>
@@
 <attribute name="NAME" x="88.646" y="26.543" size="1" layer="25" rot="R90"/>
 </element>
-<element name="C10" library="adafruit" package="C0805" value="18fp" x="85.09" y="44.323" smashed="yes" rot="R90">
+<element name="C10" library="adafruit" package="C0805" value="" x="85.09" y="44.323" smashed="yes" rot="R90">
 <attribute name="NAME" x="85.598" y="46.609" size="1" layer="25" rot="R90"/>
 <attribute name="VALUE" x="87.376" y="43.434" size="1.27" layer="27" rot="R90"/>
@@
 <attribute name="NAME" x="67.564" y="37.211" size="1" layer="25" rot="R90"/>
 </element>
-<element name="C7" library="adafruit" package="C0805" value="18pf" x="38.481" y="33.274" smashed="yes" rot="R90">
+<element name="C7" library="adafruit" package="C0805" value="" x="38.481" y="33.274" smashed="yes" rot="R90">
 <attribute name="NAME" x="37.465" y="32.385" size="1" layer="25" rot="R90"/>
 <attribute name="VALUE" x="40.767" y="32.385" size="1.27" layer="27" rot="R90"/>
 </element>
-<element name="C8" library="adafruit" package="C0805" value="18pf" x="41.91" y="37.084" smashed="yes">
+<element name="C8" library="adafruit" package="C0805" value="" x="41.91" y="37.084" smashed="yes">
 <attribute name="NAME" x="41.021" y="38.1" size="1" layer="25"/>
 <attribute name="VALUE" x="41.021" y="34.798" size="1.27" layer="27"/>
 </element>
-<element name="C9" library="adafruit" package="C0805" value="18pf" x="85.725" y="33.909" smashed="yes">
+<element name="C9" library="adafruit" package="C0805" value="" x="85.725" y="33.909" smashed="yes">
 <attribute name="NAME" x="84.836" y="34.925" size="1" layer="25"/>
 <attribute name="VALUE" x="84.836" y="31.623" size="1.27" layer="27"/>
