File: E-P-099-R2.5.sch (EAGLE design)
At the start: 86 parts, among them J1 AVR_ISP

Commit message: update
Parts:
- C10: value 18fp -> (none)
- C7, C8, C9: value 18pf -> (none)
Other:
- note removed: "Do not add unless needed"
Changed lines of the file:
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@@
 <part name="C5" library="adafruit" deviceset="C-US" device="C0805" value="0.1uF"/>
 <part name="R5" library="adafruit" deviceset="R-US_" device="M0805" value="1K"/>
-<part name="C7" library="adafruit" deviceset="C-US" device="C0805" value="18pf"/>
-<part name="C8" library="adafruit" deviceset="C-US" device="C0805" value="18pf"/>
+<part name="C7" library="adafruit" deviceset="C-US" device="C0805"/>
+<part name="C8" library="adafruit" deviceset="C-US" device="C0805"/>
 <part name="LED0" library="Shell2013" deviceset="LED" device="1206"/>
 <part name="R6" library="adafruit" deviceset="R-US_" device="M0805" value="1K"/>
 <part name="LED1" library="Shell2013" deviceset="LED" device="1206"/>
 <part name="R7" library="adafruit" deviceset="R-US_" device="M0805" value="1K"/>
-<part name="C9" library="adafruit" deviceset="C-US" device="C0805" value="18pf"/>
-<part name="C10" library="adafruit" deviceset="C-US" device="C0805" value="18fp"/>
+<part name="C9" library="adafruit" deviceset="C-US" device="C0805"/>
+<part name="C10" library="adafruit" deviceset="C-US" device="C0805"/>
 <part name="STANDOFF1" library="SparkFun-Electromechanical" deviceset="STAND-OFF" device=""/>
 <part name="STANDOFF2" library="SparkFun-Electromechanical" deviceset="STAND-OFF" device=""/>
@@
 <sheet>
 <plain>
-<text x="332.74" y="193.04" size="1.778" layer="91">Do not add unless needed</text>
-<text x="332.74" y="203.2" size="1.778" layer="91">Do not add unless needed</text>
 </plain>
 <instances>
