File: E-P-099-R2.8.sch (EAGLE design)
At the start: 86 parts, among them J1 AVR_ISP

Commit message: VER.3
Added through hole mosfets, fixed input switch logic, improved pull downs on inout, added connector for break switch,   increased board size and fixed routing,
Parts:
- removed JP1: (no value), SparkFun-Retired:JUMPER-2PTH
- removed U$10, U$11, U$13, U$14, U$15, U$20: SIA426DJ, Shell2013:SIA426DJ
- added Q1, Q2, Q3, Q4, Q5, Q6: BSS101, transistor-fet:BSS101
- added U$3: TE770966, Shell2013(1):TE770966
Connections:
- removed net N$27: FRONT.6, FRONT.8, U$10.D
- removed net N$43: REAR.4, U$14.D
- removed net N$49: LED2.A, R31.2
- new net N$14: Q2.G, R13.2
- new net N$15: Q1.G, R3.2
- new net N$22: FRONT.5, Q5.D
- net +12V: now also FRONT.1, FRONT.3, REAR.4; no longer FRONT.5, FRONT.7, REAR.5
- net +5V: now also SWITCH_PANNEL.1, SWITCH_PANNEL.2, SWITCH_PANNEL.3, U$3.V/SIG
- net BREAK_SWITCH: now also LED1.A, U$3.G/LOW; no longer JP1.1, LED12.A
- net DRIVING_LIGHTS_SWITCH: now also LED6.A, SWITCH_PANNEL.6; no longer LED10.A, SWITCH_PANNEL.1
- net FREE: now also LED0.A, SWITCH_PANNEL.8; no longer SWITCH_PANNEL.6
- net GND: now also Q1.S, Q2.S, Q3.S, Q4.S, Q5.S, Q6.S; no longer FRONT.SHD1, FRONT.SHD2, JP1.2, SWITCH_PANNEL.7, SWITCH_PANNEL.8, SWITCH_PANNEL.SHD1, SWITCH_PANNEL.SHD2, U$10.S, U$11.S, U$13.S, U$14.S, U$15.S, U$20.S
- net HAZ_SWITCH: now also LED10.A, SWITCH_PANNEL.7; no longer LED11.A, SWITCH_PANNEL.3
- net LEFT_SWITCH: now also LED11.A, SWITCH_PANNEL.5; no longer LED1.A, SWITCH_PANNEL.4
- net N$17: now also LED2.A, Q5.G; no longer LED2.C, U$20.G
- net N$20: now also FRONT.7, FRONT.8, Q6.D; no longer FRONT.1, U$20.D
- net N$21: now also FRONT.6, Q4.D; no longer R3.2, U$14.G
- net N$23: now also LED2.C, R31.2; no longer FRONT.3, U$11.D
- net N$33: now also Q4.G; no longer U$11.G
- net N$35: now also Q6.G; no longer U$10.G
- net N$4: now also Q3.D; no longer U$13.D
- net N$5: now also Q1.D; no longer U$15.D
- net N$7: now also Q2.D, REAR.5; no longer R13.2, U$15.G
- net N$8: now also Q3.G; no longer U$13.G
- net RIGHT_SWITCH: now also LED12.A, SWITCH_PANNEL.4; no longer LED0.A, SWITCH_PANNEL.2
- net WIPER_SWITCH: no longer LED6.A, SWITCH_PANNEL.5
Other:
- moved on the sheet: FRONT, LED0, LED1, LED10, LED11, LED12, LED2, LED3, LED4, LED6, LED7, LED9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
