File: E-P-099-R2.8.sch (EAGLE design)
At the start: 86 parts, among them J1 AVR_ISP, Q1 BSS101, Q2 BSS101, Q3 BSS101, Q4 BSS101, Q5 BSS101, Q6 BSS101

Commit message: added pull down resistors to switches, added windshield wiper switch, added capacitors to make mike happy, adjusted led circuit on outputs might need different resistor values, changed a couple other things
Parts:
- removed C17: 100uF, SparkFun-Capacitors:47UF-50V-20%(ELECT)
- removed U$18: CRYSTAL, mylibrary:CRYSTAL
- added C1, C2: 100UF-POLAR, 100uF_Cap:100UF-POLAR
- added LED13, LED14, LED15: (no value), led:LEDCHIPLED_0805
- added LED16: (no value), SparkFun-LED:LED0603
- added R10, R11, R15, R25, R35, R9: 10K, resistor:R-US_R0805
- added R26, R28, R29, R40: 1K, SparkFun-Passives:RESISTOR0805-RES
- added R30: 430, SparkFun-Passives:RESISTOR0805-RES
- added U$5: TE770966, Shell2013(1):TE770966
- added Y1: (no value), SparkFun-FreqCtrl:CRYSTALHC49US
- R31, R32: value 330 -> 430
- R33: value 330 -> 10K; device SparkFun-Passives:RESISTOR0805-RES -> resistor:R-US_R0805
Connections:
- removed net N$31: LED4.C, R32.2
- removed net N$38: LED3.C, R33.2
- new net N$18: LED4.A, R32.2
- new net N$24: C8.1, Y1.2
- new net N$27: LED2.A, R30.2
- new net N$28: LED16.C, R40.2
- new net N$32: LED13.A, R26.2
- new net N$34: LED14.A, R28.1
- new net N$36: LED15.A, R29.2
- net +12V: now also R26.1, R28.2, R29.1, R30.1, R31.2, R32.1
- net +5V: now also C1.+, C2.+, U$5.V/SIG; no longer C17.+
- net BREAK_SWITCH: now also R35.2
- net DRIVING_LIGHTS_SWITCH: now also R11.2
- net FREE: now also R9.2
- net GND: now also C1.-, C2.-, R10.1, R11.1, R15.1, R25.1, R33.2, R35.1, R40.1, R9.1; no longer C17.-, R31.1, R32.1, R33.1
- net HAZ_SWITCH: now also R10.2
- net LEFT_SWITCH: now also R15.2
- net N$17: no longer LED2.A
- net N$20: now also LED15.C
- net N$21: now also LED14.C
- net N$22: now also LED13.C
- net N$23: now also LED3.A, R31.1; no longer LED2.C, R31.2
- net N$33: no longer LED4.A
- net N$35: no longer LED3.A
- net N$4: now also LED2.C
- net N$5: now also LED3.C
- net N$7: now also LED4.C
- net RIGHT_SWITCH: now also R25.2
- net WIPER_SWITCH: now also LED16.A, R33.1, U$5.G/LOW
- net XTAL1: no longer C8.1, U$18.P$2
- net XTAL2: now also Y1.1; no longer U$18.P$1
Other:
- moved on the sheet: LED0, LED11, LED12, LED2, LED3, LED4, LED6, R1, R2, R31, R32, R33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
