File: Horn Board/Horn Board.brd (EAGLE design)
At the start: 32.7 x 40.6 mm, 11 parts, among them K1 RELAY-SPDT-JZC-11F, T1 2N2222

Commit message: Added Connectors to horn board
Parts:
- added U$1, U$2, U$8: TE770966, Shell2013(1):2X1-MATE-N-LOCK
Connections:
- new net HORN_GND: D2.A, K1.3, U$1.CIRCUIT2
- new net INPUT: R1.2, R2.2, U$2.CIRCUIT2
- net GND: now also U$8.CIRCUIT2; no longer D2.A, K1.3, R1.2, R2.2
- net VCC: now also U$1.CIRCUIT1, U$2.CIRCUIT1, U$8.CIRCUIT1
Routing:
- net GND: track 48.0 -> 13.9 mm
Changed lines of the file:
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@@
 <?xml version="1.0" encoding="utf-8"?>
 <!DOCTYPE eagle SYSTEM "eagle.dtd">
-<eagle version="8.3.2">
+<eagle version="8.4.1">
 <drawing>
 <settings>
@@
 <layers>
 <layer number="1" name="Top" color="4" fill="1" visible="yes" active="yes"/>
+<layer number="2" name="Route2" color="1" fill="3" visible="no" active="no"/>
+<layer number="3" name="Route3" color="4" fill="3" visible="no" active="no"/>
+<layer number="14" name="Route14" color="1" fill="6" visible="no" active="no"/>
+<layer number="15" name="Route15" color="4" fill="6" visible="no" active="no"/>
 <layer number="16" name="Bottom" color="1" fill="1" visible="yes" active="yes"/>
 <layer number="17" name="Pads" color="2" fill="1" visible="yes" active="yes"/>
@@
 <param name="dpMaxLengthDifference" value="10mm"/>
 <param name="dpGapFactor" value="2.5"/>
-<param name="checkGrid" value="0"/>
 <param name="checkAngle" value="0"/>
 <param name="checkFont" value="1"/>
 <param name="checkRestrict" value="1"/>
+<param name="checkStop" value="0"/>
 <param name="useDiameter" value="13"/>
 <param name="maxErrors" value="50"/>
@@
 <element name="H3" library="SparkFun-Hardware" library_urn="urn:adsk.eagle:library:519" package="STAND-OFF" package3d_urn="urn:adsk.eagle:package:38630/1" value="STAND-OFF" x="29.21" y="31.75"/>
 <element name="H4" library="SparkFun-Hardware" library_urn="urn:adsk.eagle:library:519" package="STAND-OFF" package3d_urn="urn:adsk.eagle:package:38630/1" value="STAND-OFF" x="3.81" y="64.77"/>
+<element name="U$8" library="Shell2013(1)" package="2X1-MATE-N-LOCK" value="TE770966" x="6.35" y="-1.27"/>
+<element name="U$1" library="Shell2013(1)" package="2X1-MATE-N-LOCK" value="TE770966" x="6.35" y="-27.94"/>
+<element name="U$2" library="Shell2013(1)" package="2X1-MATE-N-LOCK" value="TE770966" x="6.35" y="-54.61"/>
 </elements>
 <signals>
@@
 <wire x1="8.9916" y1="53.34" x2="8.9916" y2="62.1792" width="0.1524" layer="1"/>
 <wire x1="8.9916" y1="62.1792" x2="8.89" y2="62.23" width="0.1524" layer="1"/>
+<contactref element="U$8" pad="CIRCUIT1"/>
+<contactref element="U$1" pad="CIRCUIT1"/>
+<contactref element="U$2" pad="CIRCUIT1"/>
+<wire x1="4.28" y1="12.96" x2="6.35" y2="53.34" width="0" layer="19" extent="1-1"/>
+<wire x1="4.28" y1="-13.71" x2="4.28" y2="12.96" width="0" layer="19" extent="1-1"/>
+<wire x1="4.28" y1="-40.38" x2="4.28" y2="-13.71" width="0" layer="19" extent="1-1"/>
 </signal>
 <signal name="GND">
-<contactref element="D2" pad="A"/>
-<contactref element="K1" pad="3"/>
 <contactref element="K1" pad="2"/>
 <contactref element="LED1" pad="C@1"/>
 <contactref element="T1" pad="C"/>
-<contactref element="R1" pad="2"/>
-<contactref element="R2" pad="2"/>
 <wire x1="29.1084" y1="49.53" x2="29.1084" y2="50.7492" width="0.1524" layer="1"/>
 <wire x1="22.86" y1="43.2816" x2="26.5176" y2="46.9392" width="0.1524" layer="1"/>
@@
 <wire x1="29.1084" y1="50.7492" x2="29.21" y2="50.8" width="0.1524" layer="1"/>
 <wire x1="22.86" y1="43.2816" x2="22.86" y2="43.18" width="0.1524" layer="1"/>
-<wire x1="17.8308" y1="31.6992" x2="17.8308" y2="30.48" width="0.1524" layer="1"/>
-<wire x1="22.86" y1="36.7284" x2="17.8308" y2="31.6992" width="0.1524" layer="1"/>
-<wire x1="22.86" y1="38.1" x2="22.86" y2="36.7284" width="0.1524" layer="1"/>
-<wire x1="17.8308" y1="30.48" x2="17.78" y2="30.48" width="0.1524" layer="1"/>
-<wire x1="22.86" y1="38.1" x2="27.94" y2="38.1" width="0.1524" layer="1"/>
-<wire x1="11.43" y1="38.1" x2="6.35" y2="38.1" width="0.1524" layer="1"/>
-<wire x1="17.8308" y1="31.6992" x2="11.43" y2="38.1" width="0.1524" layer="1"/>
-<wire x1="22.86" y1="38.1" x2="22.86" y2="43.18" width="0.1524" layer="1"/>
 <wire x1="28.6512" y1="44.8056" x2="29.1084" y2="44.8056" width="0.1524" layer="1"/>
 <wire x1="26.5176" y1="46.9392" x2="28.6512" y2="44.8056" width="0.1524" layer="1"/>
@@
 <vertex x="0" y="27.94"/>
 </polygon>
+<contactref element="U$8" pad="CIRCUIT2"/>
+<wire x1="8.42" y1="12.96" x2="22.86" y2="43.18" width="0" layer="19" extent="1-1"/>
 </signal>
 <signal name="N$2">
@@
 <wire x1="29.21" y1="39.37" x2="30.48" y2="38.1" width="0.1524" layer="1"/>
 </signal>
+<signal name="INPUT">
+<contactref element="R1" pad="2"/>
+<contactref element="R2" pad="2"/>
+<contactref element="U$2" pad="CIRCUIT2"/>
+<wire x1="17.78" y1="30.48" x2="27.94" y2="38.1" width="0" layer="19" extent="1-1"/>
+<wire x1="8.42" y1="-40.38" x2="17.78" y2="30.48" width="0" layer="19" extent="1-1"/>
+</signal>
+<signal name="HORN_GND">
+<contactref element="K1" pad="3"/>
+<contactref element="D2" pad="A"/>
+<contactref element="U$1" pad="CIRCUIT2"/>
+<wire x1="6.35" y1="38.1" x2="22.86" y2="38.1" width="0" layer="19" extent="1-1"/>
+<wire x1="8.42" y1="-13.71" x2="6.35" y2="38.1" width="0" layer="19" extent="1-1"/>
+</signal>
 </signals>
