File: Horn Board/Horn Board Rev 1.brd (EAGLE design)
At the start: 50 x 50 mm, 14 parts, among them K1 RELAY-SPDT-JZC-11F, T1 2N2222

Commit message: Gerbers Generated
Parts:
- moved U$2 14.5 mm to (52.2, 35.6), turned to 90 degrees
- moved U$8 10.9 mm to (-3.36, 27.2), turned to 270 degrees
- moved U$1 5.00 mm to (52.0, 13.8)
Routing:
- net HORN_GND: track 18.1 -> 28.0 mm
- net GND: track 44.9 -> 39.8 mm
- net N$1: track 15.8 -> 11.8 mm
- net VCC: track 95.3 -> 94.5 mm
Other:
- board text added: "HORN"
- board text added: "PWR IN"
- board text added: "WHEEL"
Changed lines of the file:
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@@
 <?xml version="1.0" encoding="utf-8"?>
 <!DOCTYPE eagle SYSTEM "eagle.dtd">
-<eagle version="8.3.2">
+<eagle version="8.4.1">
 <drawing>
 <settings>
@@
 <wire x1="50" y1="50" x2="0" y2="50" width="0" layer="20"/>
 <wire x1="0" y1="50" x2="0" y2="0" width="0" layer="20"/>
+<text x="1" y="19" size="1.778" layer="21">PWR IN</text>
+<text x="40" y="20" size="1.778" layer="21">HORN</text>
+<text x="40" y="27" size="1.778" layer="21">WHEEL</text>
 </plain>
 <attributes>
@@
 <param name="dpMaxLengthDifference" value="10mm"/>
 <param name="dpGapFactor" value="2.5"/>
-<param name="checkGrid" value="0"/>
 <param name="checkAngle" value="0"/>
 <param name="checkFont" value="1"/>
 <param name="checkRestrict" value="1"/>
+<param name="checkStop" value="0"/>
 <param name="useDiameter" value="13"/>
 <param name="maxErrors" value="50"/>
@@
 <element name="R2" library="adafruit" library_urn="urn:adsk.eagle:library:420" package="0204V" value="1k" x="14.7" y="46.53"/>
 <element name="T1" library="adafruit" library_urn="urn:adsk.eagle:library:420" package="TO92-EBC-OVAL" value="2N2222" x="10.63" y="37.95" rot="R180"/>
-<element name="U$1" library="Shell2013(1)" package="2X1-MATE-N-LOCK" value="TE770966" x="47.02" y="13.77" rot="R90"/>
-<element name="U$2" library="Shell2013(1)" package="2X1-MATE-N-LOCK" value="TE770966" x="42.59" y="24.77"/>
-<element name="U$8" library="Shell2013(1)" package="2X1-MATE-N-LOCK" value="TE770966" x="6.22" y="32.36" rot="R180"/>
+<element name="U$1" library="Shell2013(1)" package="2X1-MATE-N-LOCK" value="TE770966" x="52.02" y="13.77" rot="R90"/>
+<element name="U$2" library="Shell2013(1)" package="2X1-MATE-N-LOCK" value="TE770966" x="52.23" y="35.59" rot="R90"/>
+<element name="U$8" library="Shell2013(1)" package="2X1-MATE-N-LOCK" value="TE770966" x="-3.36" y="27.22" rot="R270"/>
 </elements>
 <signals>
@@
 <contactref element="U$1" pad="CIRCUIT1"/>
 <contactref element="U$2" pad="CIRCUIT1"/>
-<wire x1="35.2044" y1="38.862" x2="40.386" y2="38.862" width="1" layer="1"/>
-<wire x1="32.6136" y1="36.2712" x2="35.2044" y2="38.862" width="1" layer="1"/>
-<wire x1="40.386" y1="38.862" x2="40.52" y2="39" width="1" layer="1"/>
-<wire x1="32.6136" y1="36.2712" x2="32.56" y2="36.17" width="1" layer="1"/>
-<wire x1="11.7348" y1="18.1356" x2="8.382" y2="18.1356" width="1" layer="16"/>
-<wire x1="17.2212" y1="23.622" x2="11.7348" y2="18.1356" width="1" layer="16"/>
-<wire x1="8.382" y1="18.1356" x2="8.29" y2="18.13" width="1" layer="16"/>
-<wire x1="17.2212" y1="23.622" x2="17.25" y2="23.68" width="0.1524" layer="16"/>
 <wire x1="29.2608" y1="11.7348" x2="32.766" y2="11.7348" width="1" layer="16"/>
-<wire x1="17.3736" y1="18.622" x2="22.5928" y2="16.4028" width="1" layer="16"/>
+<wire x1="22.5928" y1="16.4028" x2="17.3736" y2="18.622" width="1" layer="16"/>
 <wire x1="22.5928" y1="16.4028" x2="29.2608" y2="11.7348" width="1" layer="16"/>
-<wire x1="32.766" y1="11.7348" x2="32.79" y2="11.7" width="1" layer="16"/>
+<wire x1="32.766" y1="11.7348" x2="37.79" y2="11.7" width="1" layer="16"/>
 <wire x1="17.3736" y1="18.622" x2="17.25" y2="23.68" width="1" layer="16"/>
-<wire x1="9.4488" y1="6.644" x2="9.4488" y2="3.5052" width="1" layer="1"/>
-<wire x1="4.5772" y1="9.0156" x2="9.4488" y2="6.644" width="1" layer="1"/>
-<wire x1="4.5772" y1="13.8308" x2="4.5772" y2="9.0156" width="1" layer="1"/>
-<wire x1="8.2296" y1="17.9832" x2="4.5772" y2="13.8308" width="1" layer="1"/>
-<wire x1="9.4488" y1="3.5052" x2="9.56" y2="3.39" width="1" layer="1"/>
-<wire x1="8.2296" y1="17.9832" x2="8.29" y2="18.13" width="1" layer="1"/>
 <wire x1="28.7452" y1="20.9028" x2="28.9612" y2="32.1188" width="1" layer="16"/>
 <wire x1="22.5928" y1="16.4028" x2="28.7452" y2="20.9028" width="1" layer="16"/>
 <wire x1="28.9612" y1="32.1188" x2="32.56" y2="36.17" width="1" layer="16"/>
 <wire x1="22.5928" y1="16.4028" x2="17.25" y2="23.68" width="1" layer="16"/>
+<wire x1="32.56" y1="36.17" x2="35.35" y2="36.17" width="1.27" layer="1"/>
+<wire x1="35.35" y1="36.17" x2="38" y2="33.52" width="1.27" layer="1"/>
+<wire x1="17.25" y1="23.68" x2="11.64" y2="29.29" width="1.27" layer="1"/>
+<wire x1="11.64" y1="29.29" x2="10.87" y2="29.29" width="1.27" layer="1"/>
+<wire x1="9.56" y1="3.39" x2="17.7896" y2="11.6196" width="1.27" layer="16"/>
+<wire x1="17.7896" y1="11.6196" x2="17.7896" y2="11.8096" width="1.27" layer="16"/>
+<wire x1="17.7896" y1="11.8096" x2="22.3828" y2="16.4028" width="1.27" layer="16"/>
+<wire x1="22.3828" y1="16.4028" x2="22.5928" y2="16.4028" width="1.27" layer="16"/>
 </signal>
 <signal name="GND">
@@
 <contactref element="T1" pad="C"/>
 <contactref element="U$8" pad="CIRCUIT2"/>
-<wire x1="6.096" y1="37.1856" x2="3.048" y2="37.1856" width="1" layer="1"/>
-<wire x1="3.048" y1="37.1856" x2="2.286" y2="37.1856" width="1" layer="1"/>
-<wire x1="8.0772" y1="39.1668" x2="6.096" y2="37.1856" width="1" layer="1"/>
-<wire x1="2.286" y1="37.1856" x2="2.24" y2="37.04" width="1" layer="1"/>
-<wire x1="8.0772" y1="39.1668" x2="8.09" y2="39.22" width="1" layer="1"/>
-<wire x1="3.048" y1="19.2024" x2="3.048" y2="37.1856" width="1" layer="1"/>
-<wire x1="4.1148" y1="18.1356" x2="3.048" y2="19.2024" width="1" layer="1"/>
-<wire x1="4.1148" y1="18.1356" x2="4.15" y2="18.13" width="1" layer="1"/>
-<wire x1="11.43" y1="11.1252" x2="19.6596" y2="11.1252" width="1" layer="16"/>
-<wire x1="4.572" y1="17.9832" x2="11.43" y2="11.1252" width="1" layer="16"/>
-<wire x1="4.2672" y1="17.9832" x2="4.572" y2="17.9832" width="1" layer="16"/>
-<wire x1="19.6596" y1="11.1252" x2="19.72" y2="11.01" width="1" layer="16"/>
-<wire x1="4.2672" y1="17.9832" x2="4.15" y2="18.13" width="1" layer="16"/>
 <polygon width="0.1524" layer="1">
 <vertex x="0" y="50"/>
@@
 <vertex x="0" y="0"/>
 </polygon>
+<wire x1="8.09" y1="39.22" x2="8.09" y2="27.91" width="1.27" layer="1"/>
+<wire x1="8.09" y1="27.91" x2="11" y2="25" width="1.27" layer="1"/>
+<wire x1="11" y1="25" x2="11" y2="19.73" width="1.27" layer="1"/>
+<wire x1="11" y1="19.73" x2="19.72" y2="11.01" width="1.27" layer="1"/>
+<wire x1="2.24" y1="37.04" x2="5.91" y2="37.04" width="0.2" layer="1"/>
+<wire x1="5.91" y1="37.04" x2="8.09" y2="39.22" width="1.27" layer="1"/>
+<wire x1="11" y1="25" x2="10.87" y2="25.15" width="0" layer="19" extent="1-1"/>
 </signal>
 <signal name="N$2">
@@
 <wire x1="13.2588" y1="39.1668" x2="13.17" y2="39.22" width="1" layer="1"/>
 <wire x1="17.2212" y1="36.2712" x2="17.32" y2="36.17" width="0.1524" layer="1"/>
-<wire x1="9.6012" y1="28.4988" x2="9.6012" y2="11.1252" width="1" layer="1"/>
-<wire x1="17.2212" y1="36.1188" x2="9.6012" y2="28.4988" width="1" layer="1"/>
-<wire x1="9.6012" y1="11.1252" x2="9.56" y2="11.01" width="1" layer="1"/>
-<wire x1="17.2212" y1="36.1188" x2="17.32" y2="36.17" width="0.1524" layer="1"/>
+<wire x1="13.7575" y1="22.7936" x2="14" y2="22.5511" width="1.27" layer="16"/>
+<wire x1="14" y1="22.5511" x2="14" y2="16" width="1.27" layer="16"/>
+<wire x1="17.32" y1="36.17" x2="13.7575" y2="32.6075" width="1.27" layer="16"/>
+<wire x1="13.7575" y1="32.6075" x2="13.7575" y2="22.7936" width="1.27" layer="16"/>
+<wire x1="14" y1="16" x2="9.56" y2="11.56" width="1.27" layer="16"/>
+<wire x1="9.56" y1="11.56" x2="9.56" y2="11.01" width="1.27" layer="16"/>
 </signal>
 <signal name="N$5">
 <contactref element="R2" pad="1"/>
 <contactref element="LED1" pad="A@1"/>
-<wire x1="2.24" y1="38.04" x2="2.24" y2="38.74" width="1" layer="1"/>
-<wire x1="2.24" y1="38.74" x2="10" y2="46.5" width="1" layer="1"/>
+<wire x1="2.24" y1="38.04" x2="2.24" y2="38.74" width="0.2" layer="1"/>
+<wire x1="2.24" y1="38.74" x2="10" y2="46.5" width="0.2" layer="1"/>
 <wire x1="10" y1="46.5" x2="13.4" y2="46.5" width="1" layer="1"/>
 <wire x1="13.4" y1="46.5" x2="13.43" y2="46.53" width="1" layer="1"/>
@@
 <contactref element="D2" pad="A"/>
 <contactref element="U$1" pad="CIRCUIT2"/>
-<wire x1="32.766" y1="23.4696" x2="32.766" y2="15.8496" width="1" layer="1"/>
+<wire x1="32.766" y1="23.4696" x2="32.766" y2="15.8496" width="1.27" layer="1"/>
 <wire x1="32.6136" y1="23.622" x2="32.766" y2="23.4696" width="0.1524" layer="1"/>
-<wire x1="32.766" y1="15.8496" x2="32.79" y2="15.84" width="0.1524" layer="1"/>
+<wire x1="32.766" y1="15.8496" x2="37.79" y2="15.84" width="0.1524" layer="1"/>
 <wire x1="32.6136" y1="23.622" x2="32.49" y2="23.68" width="1" layer="1"/>
-<wire x1="28.194" y1="11.1252" x2="24.8412" y2="11.1252" width="1" layer="1"/>
-<wire x1="32.766" y1="15.6972" x2="28.194" y2="11.1252" width="1" layer="1"/>
+<wire x1="28.194" y1="11.1252" x2="24.8412" y2="11.1252" width="1.27" layer="1"/>
+<wire x1="32.766" y1="15.6972" x2="28.194" y2="11.1252" width="1.27" layer="1"/>
 <wire x1="24.8412" y1="11.1252" x2="24.8" y2="11.01" width="1" layer="1"/>
-<wire x1="32.766" y1="15.6972" x2="32.79" y2="15.84" width="0.1524" layer="1"/>
+<wire x1="32.766" y1="15.6972" x2="37.79" y2="15.84" width="1.27" layer="1"/>
 </signal>
 <signal name="N$1">
 <contactref element="U$2" pad="CIRCUIT2"/>
 <contactref element="R1" pad="1"/>
-<wire x1="36.576" y1="47.0916" x2="32.3088" y2="47.0916" width="1" layer="1"/>
-<wire x1="44.6532" y1="39.0144" x2="36.576" y2="47.0916" width="1" layer="1"/>
-<wire x1="32.3088" y1="47.0916" x2="32.28" y2="47.14" width="1" layer="1"/>
-<wire x1="44.6532" y1="39.0144" x2="44.66" y2="39" width="1" layer="1"/>
+<wire x1="38" y1="37.66" x2="38" y2="41.42" width="1.27" layer="1"/>
+<wire x1="38" y1="41.42" x2="32.28" y2="47.14" width="1.27" layer="1"/>
 </signal>
 </signals>
