File: Archive/E-P-099-R2.8.sch (EAGLE design)
At the start: 103 parts, among them J1 AVR_ISP, Q1 BSS101, Q2 BSS101, Q3 BSS101, Q4 BSS101, Q5 BSS101, Q6 BSS101

Commit message: added separate power for servo, cleaned up a bit of board layout, remade some missing eagle libraries and added them to library repo
Parts:
- removed JP2: (no value), E-P-099-R2.2:PINHD-2X14
- added C6, C9: 100UF-POLAR, 100uF_Cap:100UF-POLAR
- added D2: MBRA140, SparkFun-DiscreteSemi:MBRA140
- added E1: 5555140-6, 5555140-6 RJ11:5555140-6
- added U$6: TE770966, Shell2013(1):TE770966
- U$1: value TE770966 -> FUSEMINI-BLADE; device Shell2013(1):TE770966 -> Shell2013:FUSEMINI-BLADE
Connections:
- removed net N$24: C8.1, Y1.2
- new net N$29: U$1.IN, U$6.V/SIG
- new net SERVO_V: C9.+, D2.C, SERVO.2, U$1.OUT
- net +12V: now also C6.+
- net +5V: no longer SERVO.2
- net GND: now also C6.-, C9.-, D2.A, E1.1, E1.6, E1.SH1, E1.SH2, U$6.G/LOW; no longer U$1.G/LOW
- net N$6: now also E1.3, E1.4; no longer U$1.V/SIG
- net XTAL1: now also C8.1, Y1.2
